File: module-pic-40pin/module-pic-40pin.kicad_pcb (KiCad board)
At the start: 2 copper layers, 93 x 61.9 mm, 27 parts, among them J1 input_power, J2 ANALOG, J3 icsp, J4 PORTB, J5 PORTC, J6 Conn_02x04_Odd_Even, J7 RB0_CONN, J8 PORTD, SW1 reset, SW2 EXT_INT0, U1 PIC16F877A-IP, Y1 20MHz

Commit message: update module-pic-40pin.kicad_pcb
Routing:
- net GND: track 294.0 -> 301.0 mm
- net /RD1: track 89.2 -> 91.9 mm
- net +5V: track 232.6 -> 235.0 mm
- net /RC6: track 35.4 -> 37.4 mm
- net /RC4: track 45.1 -> 47.0 mm
- net /RB7: track 67.1 -> 68.2 mm
- net Net-(C1-Pad1): track 27.2 -> 28.2 mm
- net /RB0: track 81.9 -> 82.7 mm
- net /RA4: track 50.4 -> 51.2 mm
- net /RC7: track 54.4 -> 55.0 mm

Commit message: update module-pic-40pin.kicad_pcb
Routing:
- net /RA4: track 51.2 -> 53.6 mm
- net /RC6: track 37.4 -> 38.7 mm
- net /RC7: track 55.0 -> 55.8 mm
- net /RC4: track 47.0 -> 47.6 mm
Changed lines of the file:
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@@
   (segment (start 91.0336 88.2904) (end 90.1192 87.376) (width 0.3) (layer "B.Cu") (net 22))
   (segment (start 90.1192 79.5528) (end 86.702 76.1356) (width 0.3) (layer "B.Cu") (net 22))
+  (segment (start 89.242 76.415) (end 90.1954 77.3684) (width 0.3) (layer "B.Cu") (net 23))
   (segment (start 93.6244 77.3684) (end 95.6056 75.3872) (width 0.3) (layer "B.Cu") (net 23))
-  (segment (start 89.242 75.3228) (end 91.2876 77.3684) (width 0.3) (layer "B.Cu") (net 23))
-  (segment (start 91.2876 77.3684) (end 93.6244 77.3684) (width 0.3) (layer "B.Cu") (net 23))
   (segment (start 95.6056 72.9488) (end 92.0496 69.3928) (width 0.3) (layer "B.Cu") (net 23))
+  (segment (start 89.242 74.2351) (end 89.242 76.415) (width 0.3) (layer "B.Cu") (net 23))
+  (segment (start 95.6056 75.3872) (end 95.6056 72.9488) (width 0.3) (layer "B.Cu") (net 23))
+  (segment (start 63.5 69.3928) (end 62.1792 68.072) (width 0.3) (layer "B.Cu") (net 23))
   (segment (start 92.0496 69.3928) (end 63.5 69.3928) (width 0.3) (layer "B.Cu") (net 23))
-  (segment (start 95.6056 75.3872) (end 95.6056 72.9488) (width 0.3) (layer "B.Cu") (net 23))
-  (segment (start 89.242 74.2351) (end 89.242 75.3228) (width 0.3) (layer "B.Cu") (net 23))
-  (segment (start 63.5 69.3928) (end 62.1792 68.072) (width 0.3) (layer "B.Cu") (net 23))
-  (segment (start 90.5257 71.6788) (end 63.246 71.6788) (width 0.3) (layer "B.Cu") (net 24))
-  (segment (start 91.782 72.9351) (end 90.5257 71.6788) (width 0.3) (layer "B.Cu") (net 24))
+  (segment (start 90.1954 77.3684) (end 93.6244 77.3684) (width 0.3) (layer "B.Cu") (net 23))
   (segment (start 91.782 74.2351) (end 91.782 72.9351) (width 0.3) (layer "B.Cu") (net 24))
-  (segment (start 63.246 71.6788) (end 62.1792 70.612) (width 0.3) (layer "B.Cu") (net 24))
-  (segment (start 90.4748 73.0504) (end 90.4748 75.2856) (width 0.3) (layer "B.Cu") (net 25))
-  (segment (start 84.112971 72.4916) (end 89.916 72.4916) (width 0.3) (layer "B.Cu") (net 25))
-  (segment (start 91.4908 76.3016) (end 93.2688 76.3016) (width 0.3) (layer "B.Cu") (net 25))
-  (segment (start 62.992 73.9648) (end 82.639771 73.9648) (width 0.3) (layer "B.Cu") (net 25))
-  (segment (start 82.639771 73.9648) (end 84.112971 72.4916) (width 0.3) (layer "B.Cu") (net 25))
-  (segment (start 93.2688 76.3016) (end 94.322 75.2484) (width 0.3) (layer "B.Cu") (net 25))
-  (segment (start 89.916 72.4916) (end 90.4748 73.0504) (width 0.3) (layer "B.Cu") (net 25))
-  (segment (start 90.4748 75.2856) (end 91.4908 76.3016) (width 0.3) (layer "B.Cu") (net 25))
+  (segment (start 62.3824 70.8152) (end 62.1792 70.612) (width 0.3) (layer "B.Cu") (net 24))
+  (segment (start 91.782 72.9351) (end 89.6621 70.8152) (width 0.3) (layer "B.Cu") (net 24))
+  (segment (start 89.6621 70.8152) (end 62.3824 70.8152) (width 0.3) (layer "B.Cu") (net 24))
+  (segment (start 90.4748 76.073) (end 91.0336 76.6318) (width 0.3) (layer "B.Cu") (net 25))
+  (segment (start 89.2556 71.8312) (end 90.4748 73.0504) (width 0.3) (layer "B.Cu") (net 25))
+  (segment (start 90.4748 73.0504) (end 90.4748 76.073) (width 0.3) (layer "B.Cu") (net 25))
+  (segment (start 82.9564 71.8312) (end 89.2556 71.8312) (width 0.3) (layer "B.Cu") (net 25))
+  (segment (start 94.322 75.2484) (end 94.322 74.2351) (width 0.3) (layer "B.Cu") (net 25))
+  (segment (start 92.9386 76.6318) (end 94.322 75.2484) (width 0.3) (layer "B.Cu") (net 25))
+  (segment (start 91.0336 76.6318) (end 92.9386 76.6318) (width 0.3) (layer "B.Cu") (net 25))
+  (segment (start 80.8228 73.9648) (end 82.9564 71.8312) (width 0.3) (layer "B.Cu") (net 25))
+  (segment (start 62.992 73.9648) (end 80.8228 73.9648) (width 0.3) (layer "B.Cu") (net 25))
   (segment (start 62.1792 73.152) (end 62.992 73.9648) (width 0.3) (layer "B.Cu") (net 25))
-  (segment (start 94.322 75.2484) (end 94.322 74.2351) (width 0.3) (layer "B.Cu") (net 25))
+  (segment (start 92.3036 81.0768) (end 92.3036 89.8652) (width 0.3) (layer "B.Cu") (net 26))
+  (segment (start 96.862 76.5184) (end 92.3036 81.0768) (width 0.3) (layer "B.Cu") (net 26))
   (segment (start 62.992 76.5048) (end 62.1792 75.692) (width 0.3) (layer "B.Cu") (net 26))
+  (segment (start 92.3036 89.8652) (end 91.7448 90.424) (width 0.3) (layer "B.Cu") (net 26))
   (segment (start 87.2236 86.9188) (end 76.8096 76.5048) (width 0.3) (layer "B.Cu") (net 26))
+  (segment (start 87.2236 90.043) (end 87.2236 86.9188) (width 0.3) (layer "B.Cu") (net 26))
+  (segment (start 87.6046 90.424) (end 87.2236 90.043) (width 0.3) (layer "B.Cu") (net 26))
+  (segment (start 96.862 74.2351) (end 96.862 76.5184) (width 0.3) (layer "B.Cu") (net 26))
   (segment (start 76.8096 76.5048) (end 62.992 76.5048) (width 0.3) (layer "B.Cu") (net 26))
-  (segment (start 92.3036 89.2048) (end 91.0844 90.424) (width 0.3) (layer "B.Cu") (net 26))
-  (segment (start 88.392 90.424) (end 87.2236 89.2556) (width 0.3) (layer "B.Cu") (net 26))
-  (segment (start 96.862 74.2351) (end 96.862 76.5184) (width 0.3) (layer "B.Cu") (net 26))
-  (segment (start 96.862 76.5184) (end 92.3036 81.0768) (width 0.3) (layer "B.Cu") (net 26))
-  (segment (start 87.2236 89.2556) (end 87.2236 86.9188) (width 0.3) (layer "B.Cu") (net 26))
-  (segment (start 91.0844 90.424) (end 88.392 90.424) (width 0.3) (layer "B.Cu") (net 26))
-  (segment (start 92.3036 81.0768) (end 92.3036 89.2048) (width 0.3) (layer "B.Cu") (net 26))
+  (segment (start 91.7448 90.424) (end 87.6046 90.424) (width 0.3) (layer "B.Cu") (net 26))
   (segment (start 99.402 76.9248) (end 99.402 74.2351) (width 0.3) (layer "B.Cu") (net 27))
   (segment (start 93.5736 88.2904) (end 93.5736 82.7532) (width 0.3) (layer "B.Cu") (net 27))
@@
   (segment (start 98.3996 51.3588) (end 96.478856 51.3588) (width 0.3) (layer "B.Cu") (net 38))
   (segment (start 100.3808 53.34) (end 98.3996 51.3588) (width 0.3) (layer "B.Cu") (net 38))
-  (segment (start 128.6256 60.2488) (end 128.6256 57.785) (width 0.3) (layer "B.Cu") (net 39))
+  (segment (start 109.8296 31.3944) (end 110.24528 30.97872) (width 0.3) (layer "B.Cu") (net 39))
+  (segment (start 119.722 60.5908) (end 121.3358 62.2046) (width 0.3) (layer "B.Cu") (net 39))
+  (segment (start 110.24528 30.97872) (end 112.25872 30.97872) (width 0.3) (layer "B.Cu") (net 39))
+  (segment (start 121.3358 62.2046) (end 127.4318 62.2046) (width 0.3) (layer "B.Cu") (net 39))
+  (segment (start 127.4318 62.2046) (end 128.6256 61.0108) (width 0.3) (layer "B.Cu") (net 39))
+  (segment (start 128.6256 61.0108) (end 128.6256 57.785) (width 0.3) (layer "B.Cu") (net 39))
+  (segment (start 128.6256 57.785) (end 109.8296 38.989) (width 0.3) (layer "B.Cu") (net 39))
   (segment (start 112.25872 30.97872) (end 113.6396 32.3596) (width 0.3) (layer "B.Cu") (net 39))
   (segment (start 109.8296 38.989) (end 109.8296 31.3944) (width 0.3) (layer "B.Cu") (net 39))
-  (segment (start 109.8296 31.3944) (end 110.24528 30.97872) (width 0.3) (layer "B.Cu") (net 39))
-  (segment (start 127.9144 60.96) (end 128.6256 60.2488) (width 0.3) (layer "B.Cu") (net 39))
-  (segment (start 128.6256 57.785) (end 109.8296 38.989) (width 0.3) (layer "B.Cu") (net 39))
-  (segment (start 110.24528 30.97872) (end 112.25872 30.97872) (width 0.3) (layer "B.Cu") (net 39))
-  (segment (start 119.722 58.9951) (end 121.6869 60.96) (width 0.3) (layer "B.Cu") (net 39))
-  (segment (start 121.6869 60.96) (end 127.9144 60.96) (width 0.3) (layer "B.Cu") (net 39))
+  (segment (start 119.722 58.9951) (end 119.722 60.5908) (width 0.3) (layer "B.Cu") (net 39))
   (segment (start 120.7008 45.212) (end 118.7704 45.212) (width 0.3) (layer "B.Cu") (net 40))
   (segment (start 123.8504 48.3616) (end 120.7008 45.212) (width 0.3) (layer "B.Cu") (net 40))
